File: tl866_27c322_adapter.kicad_sch (KiCad schematic)
At the start: 11 parts, among them J1 27C322, J2 TL866_socket, Q1 MMBT3906, SW1 SW_Coded_SH-7010, SW2 SW_Push_DPDT

Commit message: Auto-commit Fri Feb 17 21:15:45 EST 2023
Other:
- company: (none) -> matei repair lab
- title: (none) -> tl866 27C* adapter
Changed lines of the file:
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@@
 (kicad_sch (version 20211123) (generator eeschema)
   (paper "A4")
+  (title_block
+    (title "tl866 27C* adapter")
+    (date "2023-02-17")
+    (rev "4.0")
+    (company "matei repair lab")
+  )
   (junction (at 55.88 75.565) (diameter 0) (color 0 0 0 0)
   )
